File: WarthoggitClone.kicad_pcb (KiCad board)
At the start: 2 copper layers, 30.5 x 49.5 mm, 52 parts, among them J1 TRIGGER_2, J10 DMS, J11 TMS, J12 HAT, J2 WEAPON_RELEASE, J3 TOP_RIGHT_SIDE, J4 PINKY_LEVER, J5 CMS_DOWN, J6 TRIGGER_1, J7 PINKY_BUTTON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

Commit message: Fix DRC
Other:
- rule trace_min: 0.2 -> 0.1524
- rule via_min_drill: 0.3 -> 0.3302
- rule via_min_size: 0.4 -> 0.6858
Changed lines of the file:
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@@
     (zone_clearance 0.254)
     (zone_45_only no)
-    (trace_min 0.2)
+    (trace_min 0.1524)
     (segment_width 0.2)
     (edge_width 0.15)
     (via_size 0.8)
     (via_drill 0.4)
-    (via_min_size 0.4)
-    (via_min_drill 0.3)
+    (via_min_size 0.6858)
+    (via_min_drill 0.3302)
     (uvia_size 0.3)
     (uvia_drill 0.1)
@@
     (pcbplotparams
       (layerselection 0x010fc_ffffffff)
-      (usegerberextensions false)
+      (usegerberextensions true)
       (usegerberattributes false)
       (usegerberadvancedattributes false)
@@
       (outputformat 1)
       (mirror false)
-      (drillshape 1)
+      (drillshape 0)
       (scaleselection 1)
-      (outputdirectory ""))
+      (outputdirectory "Gerbers/"))
   )
   (net 0 "")
