File: 2-Layer/WarthoggitClone.kicad_pcb (KiCad board)
At the start: 2 copper layers, 30.5 x 49.5 mm, 52 parts, among them J1 TRIGGER_2, J10 DMS, J11 TMS, J12 HAT, J2 WEAPON_RELEASE, J3 TOP_RIGHT_SIDE, J4 PINKY_LEVER, J5 CMS_DOWN, J6 TRIGGER_1, J7 PINKY_BUTTON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

Commit message: Split files into folders, fix missing 3D model in picoblade footprints
Other:
- rule trace_min: 0.2 -> 0.1524
- rule via_min_drill: 0.3 -> 0.3302
- rule via_min_size: 0.4 -> 0.6858
